File: Reports/Testing.kicad_sch (KiCad schematic)
At the start: 43 parts, among them J1 39303057, J2 39303057, J3 2-215307-0, J4 2-215307-0, J5 691137710002, J6 691137710002, Q1 IRF9540NPBF, U1 25AA640AT-I/SN, U2 TPS79633DCQR, U3 PC817X3NSZ1B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

Commit message: Add files via upload
Adding an updated version of the schematic and gerber file.
Parts:
- removed Q1: IRF9540NPBF, IRF9540NPBF:TO254P1052X465X1989-3, symbol IRF9540NPBF:IRF9540NPBF
- removed R14, R15: FMP100JR-52-1K2, FMP100JR_52_1K2:FMP100JR_52_1K2, symbol FMP100JR_52_1K2:FMP100JR-52-1K2
- added C4: C333C104F5G5TA, C333C104F5G5TA:C333C104F5G5TA, symbol C333C104F5G5TA:C333C104F5G5TA
- added C5: UKL2A010KDD, UKL2A010KDD:UKL2A010KDD, symbol UKL2A010KDD:UKL2A010KDD
- added H1, H2, H3, H4, H5: MountingHole_Pad, MountingHole:MountingHole_5.3mm_M5_ISO7380_Pad_TopBottom, symbol Mechanical:MountingHole_Pad
- added R14, R15: RSMF1JT2K00, FMP100JR_52_100R:FMP100JR_52_100R, symbol RSMF1JT2K00:RSMF1JT2K00
- added R18: RSF100JB-73-2R, FMP100JR_52_100R:RSF100JB_73_2R, symbol RSF100JB_73_2R:RSF100JB-73-2R
- added R19: FMP100JR-52-100R, FMP100JR_52_100R:FMP100JR_52_100R, symbol FMP100JR_52_100R:FMP100JR-52-100R
- added R20: LR1F240R, LR1F240R:LR1F240R, symbol LR1F240R:LR1F240R
- added R21: MRS25000C1651FCT00, MRS25000C1651FCT00:MRS25000C1651FCT00, symbol MRS25000C1651FCT00:MRS25000C1651FCT00
- added R22: CMF5530R000FHEB, CMF5530R000FHEB:CMF5530R000FHEB, symbol CMF5530R000FHEB:CMF5530R000FHEB
- added U7: LM317HVT/NOPB, LM317HVT_NOPB:LM317HVT_NOPB, symbol LM317HVT_NOPB:LM317HVT_NOPB
- added U8: IRF4905PBF, IRF4905PBF:IRF4905PBF, symbol IRF4905PBF:IRF4905PBF
Connections:
- net Gnd: now also C4.2, C5.2, H1.1, H2.1, H3.1, H4.1, H5.1, R22.2; no longer J1.2, R3.1
- net PWM_Out: now also R14.1
- net Tach_Out: now also R15.1
- net Vin: now also J2.1, U8.3 (D)
- net Vin_Pol: now also C4.1, R14.2, U7.3 (IN), U8.2 (S); no longer J2.1
- net Vo+_3.3V: now also R18.2; no longer LCD1.15 (A)
- net Vo-: now also R19.1
- net at D2.2, R1.2: now also U8.1 (G)
- new net: R21.2, R22.1
- new net: LCD1.15 (A), R18.1, R19.2
- new net: R20.2, R21.1, U7.1 (ADJ)
- new net Tach_In: J1.2, R3.1
- new net Vo+_10V: C5.1, R15.2, R20.1, U7.2 (OUT)
Other:
- note added: "Tach Linear Voltage Regulator"
- moved on the sheet: D2, R1, R16, R17, U5, U6
